Commit message: fix: UR5e 파지 튜닝 — 개구 단위버그·ready 포즈·플래너 폴백·드롭 클리어런스 (0/5→4/5)
5de9cb0(등록 시스템)의 후속 튜닝. 등록만으로는 UR5e 가 파지에 실패(0/5)했는데,
아래 4건을 잡아 4/5(FR3 기준 3/5 상회)까지 끌어올렸다. FR3 는 전부 불변.

핵심 수정
- 드롭 클리어런스: DROP_Z(놓는 순간 TCP 높이)를 프로파일에서 주입(apply_profile).
  Robotiq 은 프랑카보다 손끝이 길어 0.040 이면 손끝이 드롭 통 벽(25mm) 안에 박혀
  놓은 뒤 자세가 start-in-collision → 이후 계획 전부 즉시 거부. fr3=0.040,
  ur5e=0.075(손끝이 통 벽 위로 확실히 넘어감).
- 관절 목표 플래너 폴백: plan_viz_execute_joint 이 이제 pose 목표처럼
  planner_fallback 을 순차 시도한다. ready 복귀·접근처럼 통 사이를 가로지르는
  관절 이동이 기본 RRTConnect 한 방에 'Unable to solve' 로 잘리던 문제 해소.
  첫 성공 채택이라 성공 케이스(FR3 포함) 동작은 사실상 불변.
- schema: WorkspaceSpec 에 drop_z 슬롯 추가(선택, 생략 시 FR3 기준 0.040).

프로파일 값
- fr3.yaml / ur5e_robotiq85.yaml: workspace.drop_z 추가(유도 주석 포함).
- ur5e_robotiq85.srdf.xacro: 'ready' group_state 를 워크스페이스 실측으로 재튜닝
  (TCP=(0.40,0,0.30) 하향, IK elbow-up 시드 → FK 검증). 벤더 제네릭 home 은
  통에서 멀어 RRTConnect 가 ready→접근을 못 풀었다.

테스트 결정성
- test_config_profile_regression: 각 테스트 전에 fr3 프로파일을 고정하는
  autouse _pin_fr3 픽스처 추가. 활성 모델이 무엇이든 FR3 회귀가 결정적.

검증: pytest 161 passed, Gazebo 라이브 4/5 성공(bolt_3 만 하강 ~1mm 부족 —
등록/드롭과 무관한 별개 Cartesian 이슈). FR3 회귀 수치 완전 동일.

Co-Authored-By: Claude Opus 4.8 <noreply@anthropic.com>

File: src/bin_picking/srdf/ur5e_robotiq85.srdf.xacro (robot description, xacro)
@@ -27,12 +27,22 @@
            tip_link="$(arg tf_prefix)grasp_tcp"/>
   </group>
-  <!-- Ready 자세. UR 순정 `home` 과 같은 관절값을 쓴다(그룹만 다름). -->
+  <!-- Ready 자세 — 빈피킹 워크스페이스 전용(순정 home 과 다름).
+       [왜 바꿨나] 순정 home(shoulder_lift=-90°, elbow=0)은 픽 통(0.40,0.00)에서
+       멀리 떨어진 일반 대기자세라, 거기서 통 위 접근자세로 가는 관절경로를
+       RRTConnect 가 15s×10 안에 못 찾아(‘Unable to solve’) 접근 자체가 실패했다.
+       (개구·IK 는 정상이었다 — 순수 '두 유효자세 사이 계획' 실패였다.)
+       [값 유도] compute_ik 로 TCP=(0.40,0.00,0.30) '아래로 향함'을 elbow-up 시드로
+       풀어 얻은 해(관절 한계 최소여유 1.36rad)를 주값 범위로 정규화한 것.
+       shoulder_pan≈0 이라 팔이 통 쪽(+X)을 자연스럽게 향하고, 접근자세와 같은
+       IK 분기·근방에 있어 통 위 접근이 작은 관절이동으로 풀린다.
+       ※ 다른 팔 등록 시엔 이 값이 아니라 '그 팔로 통 위를 향하는' 자세를
+         같은 방식(measure_workspace/compute_ik)으로 다시 구해 넣어야 한다. -->
   <group_state name="ready" group="bin_picking_arm">
-    <joint name="$(arg tf_prefix)shoulder_pan_joint" value="0"/>
-    <joint name="$(arg tf_prefix)shoulder_lift_joint" value="-1.5707"/>
-    <joint name="$(arg tf_prefix)elbow_joint" value="0"/>
-    <joint name="$(arg tf_prefix)wrist_1_joint" value="-1.5707"/>
-    <joint name="$(arg tf_prefix)wrist_2_joint" value="0"/>
-    <joint name="$(arg tf_prefix)wrist_3_joint" value="0"/>
+    <joint name="$(arg tf_prefix)shoulder_pan_joint" value="-0.340"/>
+    <joint name="$(arg tf_prefix)shoulder_lift_joint" value="-1.364"/>
+    <joint name="$(arg tf_prefix)elbow_joint" value="1.478"/>
+    <joint name="$(arg tf_prefix)wrist_1_joint" value="1.457"/>
+    <joint name="$(arg tf_prefix)wrist_2_joint" value="1.571"/>
+    <joint name="$(arg tf_prefix)wrist_3_joint" value="1.231"/>
   </group_state>
   <!-- ============ 그리퍼 ============ -->
