Commit message: refactor: 로봇쪽 테스트 비전/카메라 제거 — 인식은 데스크톱앱 몫
볼트 인식(카메라→포인트클라우드→랭킹)은 데스크톱앱(별도 팀)이 담당하는
별개 파이프라인이다. 로봇은 데스크톱이 보낸 좌표(PICK_BOLT→/next_bolt_pose)를
받아 집기만 한다. 로봇쪽 카메라/비전은 데스크톱앱 없이 E2E를 돌려보려던
비계(scaffolding)였으므로 제거한다.

삭제:
- bolt_vision.py, vision_verify.py (비전 노드)
- launch/vision_pipeline.launch.py (gz→ROS 카메라 브릿지)
- FR3·UR5e URDF xacro 의 카메라 링크/rgbd_camera 센서
- worlds/robot_view.sdf 의 gz-sim-sensors-system 플러그인
- setup.py entry_points 2개 (bolt_vision, vision_verify)

유지(정식 입력 통로): /next_bolt_pose(EXT_POSE_TOPIC), sensing 의 외부 pose
콜백 + Gazebo pose 폴백, desktop_bridge, protocol.

문서 반영: README(파이프라인 다이어그램·모듈 지도·실행법), PROGRESS,
AGENTS.md 5개.

Co-Authored-By: Claude Opus 4.8 <noreply@anthropic.com>

File: src/bin_picking/urdf/fr3_gazebo.urdf.xacro (robot description, xacro)
@@ -27,48 +27,3 @@
   <gazebo reference="fr3_leftfinger"><gravity>false</gravity></gazebo>
   <gazebo reference="fr3_rightfinger"><gravity>false</gravity></gazebo>
-  <!-- ================= 빈피킹 비전 카메라 (eye-to-hand) =================
-    집는 통(base 기준 x=0.40, z=0) 위 0.60m 에 RGB-D 카메라를 base(fr3_link0)에
-    고정한다. 아래를 내려다보며 통 안 볼트를 스캔한다. base 에 고정이라 카메라↔
-    base TF 가 robot_state_publisher 로 자동 발행되어, perception 노드가 tf2 로
-    포인트클라우드를 base 프레임으로 변환할 수 있다.
-    ⚠ Gazebo Harmonic 의 optical_frame_id 는 포인트클라우드 좌표계를 실제로
-      회전시키지 않고 헤더 frame_id 만 바꿔 TF 불일치를 일으킨다. 데이터가
-      camera_link 좌표(x-forward)로 나오므로 frame_id 도 camera_link 여야 맞다.
-      camera_optical_link 프레임은 다른 소비자용으로 TF 트리에 남겨 둔다.     -->
-  <!-- ⚠ visual/collision 없는 '순수 프레임' — MoveIt 이 카메라 박스를 충돌체로
-       잡아 통 위 팔 자세(롤아웃)를 전부 막던 문제를 없앤다. gz rgbd_camera 센서는
-       geometry 없이 링크에 붙어도 정상 동작한다. inertial 은 gz 링크 유효성용 최소값. -->
-  <link name="camera_link">
-    <inertial>
-      <mass value="0.01"/>
-      <inertia ixx="1e-6" ixy="0" ixz="0" iyy="1e-6" iyz="0" izz="1e-6"/>
-    </inertial>
-  </link>
-  <!-- +x(gz 카메라 시선축)를 아래(-z)로: pitch +90° -->
-  <joint name="camera_joint" type="fixed">
-    <parent link="fr3_link0"/>
-    <child link="camera_link"/>
-    <origin xyz="0.40 0.0 0.60" rpy="0 1.5708 0"/>
-  </joint>
-  <!-- ROS 광학 프레임(z-forward, x-right, y-down) -->
-  <link name="camera_optical_link"/>
-  <joint name="camera_optical_joint" type="fixed">
-    <parent link="camera_link"/>
-    <child link="camera_optical_link"/>
-    <origin xyz="0 0 0" rpy="-1.5708 0 -1.5708"/>
-  </joint>
-  <gazebo reference="camera_link">
-    <sensor name="bin_camera" type="rgbd_camera">
-      <camera>
-        <horizontal_fov>1.05</horizontal_fov>       <!-- ~60°, 0.6m 에서 통 커버 -->
-        <image><width>640</width><height>480</height></image>
-        <clip><near>0.1</near><far>2.0</far></clip>
-      </camera>
-      <always_on>1</always_on>
-      <update_rate>10</update_rate>
-      <visualize>true</visualize>
-      <topic>bin_camera</topic>
-      <gz_frame_id>camera_link</gz_frame_id>
-    </sensor>
-  </gazebo>
 </robot>

File: src/bin_picking/urdf/ur5e_robotiq85_gazebo.urdf.xacro (robot description, xacro)
@@ -15,5 +15,4 @@
     world → ur_robot(UR5e) → tool0 → ur_to_robotiq 어댑터 → Robotiq 2F-85
                                                           → grasp_tcp (파지 기준)
-    base_link → camera_link (빈피킹 eye-to-hand RGB-D)
   [gz_ros2_control 주의] Robotiq 쪽은 `sim_ignition:=true` 일 때
   `ign_ros2_control/IgnitionSystem` 을 내보내는데, Jazzy 의 gz_ros2_control 이
@@ -87,38 +86,4 @@
     <origin xyz="0 0 $(arg grasp_tcp_z)" rpy="0 0 0"/>
   </joint>
-  <!-- ================== 빈피킹 비전 카메라 (eye-to-hand) ==================
-    FR3 래퍼와 같은 배치: 집는 통(base 기준 x=0.40) 위 0.60m 에서 내려다본다.
-    base 에 고정이라 카메라↔base TF 가 robot_state_publisher 로 자동 발행된다. -->
-  <link name="camera_link">
-    <inertial>
-      <mass value="0.01"/>
-      <inertia ixx="1e-6" ixy="0" ixz="0" iyy="1e-6" iyz="0" izz="1e-6"/>
-    </inertial>
-  </link>
-  <joint name="camera_joint" type="fixed">
-    <parent link="$(arg tf_prefix)base_link"/>
-    <child link="camera_link"/>
-    <origin xyz="0.40 0.0 0.60" rpy="0 1.5708 0"/>
-  </joint>
-  <link name="camera_optical_link"/>
-  <joint name="camera_optical_joint" type="fixed">
-    <parent link="camera_link"/>
-    <child link="camera_optical_link"/>
-    <origin xyz="0 0 0" rpy="-1.5708 0 -1.5708"/>
-  </joint>
-  <gazebo reference="camera_link">
-    <sensor name="bin_camera" type="rgbd_camera">
-      <camera>
-        <horizontal_fov>1.05</horizontal_fov>
-        <image><width>640</width><height>480</height></image>
-        <clip><near>0.1</near><far>2.0</far></clip>
-      </camera>
-      <always_on>1</always_on>
-      <update_rate>10</update_rate>
-      <visualize>true</visualize>
-      <topic>bin_camera</topic>
-      <gz_frame_id>camera_link</gz_frame_id>
-    </sensor>
-  </gazebo>
   <!-- ================== gz_ros2_control ================== -->
   <gazebo>
